File: KiCad/LDAD_ATOM _PRO _LCD _ABS_Enclosure_52x48_16bit.kicad_pcb (KiCad board)
At the start: 2 copper layers, 52.9 x 46.4 mm, 113 parts, among them CN3065_C2 4.7uF, CN3065_R1 1K8, CN3065_STDBY_LED1 LED, CN3965_C1 22uF, J1 TYPE-C-31-M-12, U1 MCP1525-TT, U2 ATSHA204A-MAHDA-T, U3 Battery_charger_CN3065_QFN8, U4 AHT20, U6 TEMT6000

Commit message: Add files via upload
Parts:
- added ATH20_C2: 100nF, Capacitor_SMD:C_0603_1608Metric, F.Cu at (217.5, 76.6)
- added IC_ENS1: ~, AeonLabs_Sensors:ENS160 Gas Semsor, B.Cu at (229.7, 77.4)
- added U7: BMP280, AeonLabs_Sensors:XDCR_BMP280, B.Cu at (229.7, 73.8)
- U2: footprint Package_SO:ATSHA204A Auth SOIC8 -> AeonLabs_IC:ATSHA204A-MAHDA-T UDFN-8
- moved ADC16_C1 5.38 mm to (204.2, 83.5)
- moved ADC16_C3 5.38 mm to (205.7, 83.6)
- moved ADC16_C2 5.38 mm to (204.5, 86.3)
- moved U5 5.37 mm to (202.1, 83.7)
- moved MTRT1 4.85 mm to (206.3, 89.0)
- moved MTRR1 4.74 mm to (203.6, 88.8)
- moved U6 2.72 mm to (233.0, 76.4), turned to 90 degrees
- moved U2 1.77 mm to (216.8, 86.3)
- moved I2C_SDA_R1 0.41 mm to (217.6, 79.7)
- moved IMU1 0.39 mm to (221.8, 86.6)
Routing:
- net GNDD: track 142.7 -> 178.0 mm, vias 11 -> 8
- net 3V3: track 241.5 -> 264.8 mm
- net GPIO8_I2C_SDA: track 86.6 -> 104.1 mm, vias 5 -> 6
- net GPIO9_I2C_SCL: track 86.7 -> 103.0 mm, vias 5 -> 6
- net TEMT6000_IO33: track 98.6 -> 91.4 mm
- net ADC_VOUT: track 45.7 -> 39.7 mm
- net PERIPHERALS_PWR_EN_IO10: track 33.9 -> 38.4 mm
- net (no net): track 2.74 -> 0.00 mm
- net ADC_A0: track 33.2 -> 31.0 mm
- net GND: track 318.4 -> 317.3 mm
- net VOLTAGE_REF_IO07: track 16.6 -> 15.8 mm
Other:
- board text added: "16-Bit DAQ"
- board text added: "Environment Sensors"
- board text removed: "16Bit DAQ"
- board text removed: "Luminosity Sensor"
- board text removed: "Sensor HT"

Commit message: Add files via upload
Parts:
- moved TP3 18.1 mm to (209.6, 100.8)
- moved AUR_C1 4.21 mm to (199.3, 107.4), turned to 0 degrees
- moved AUR_l1 4.19 mm to (200.2, 103.4), turned to 90 degrees
- moved PWR_FUSE1 1.92 mm to (204.3, 100.2)
- moved MTRT1 1.42 mm to (206.4, 90.4)
- moved MTRR1 1.39 mm to (203.6, 90.1)
- moved IMR1 1.04 mm to (208.1, 84.3)
- moved ADC16_C1 1.04 mm to (204.9, 84.3)
- moved ADC16_C3 1.02 mm to (206.5, 84.3)
- moved TP2 0.85 mm to (199.6, 109.5)
- moved IMR2 0.69 mm to (209.7, 84.3)
- moved AUR_R2 0.59 mm to (194.3, 105.6)
- moved AUR_R1 0.58 mm to (194.3, 107.7), turned to 180 degrees
- moved ADC16_C2 0.57 mm to (204.1, 86.6)
- moved AUR_C2 0.50 mm to (192.6, 102.7)
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Routing:
- net USB_5V0: track 65.8 -> 72.8 mm
- net Net-(AUR1-SW): track 7.29 -> 2.45 mm
- net GND: track 317.3 -> 321.8 mm, vias 21 -> 27
- net GNDD: track 178.0 -> 181.5 mm, vias 8 -> 9
- net Net-(J1-CC2): track 12.3 -> 15.2 mm
- net VIN: track 86.5 -> 88.7 mm
- net RXD0: track 46.3 -> 44.5 mm
- net TXD0: track 40.0 -> 38.2 mm
- net CHIP_EN: track 64.2 -> 62.4 mm
- net ESP_GPIO0_BOOT-DTR: track 60.7 -> 58.9 mm
- net Net-(J1-CC1): track 15.9 -> 17.6 mm
- net 3V3: track 264.8 -> 263.4 mm
- net GPIO8_I2C_SDA: track 104.1 -> 103.1 mm
- net GPIO9_I2C_SCL: track 103.0 -> 101.9 mm
- net USB_5V0F: track 32.6 -> 31.6 mm
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