File: KiCad/LDAD_ATOM _PRO _LCD _ABS_Enclosure_52x48_16bit.kicad_sch (KiCad schematic)
At the start: 86 parts, among them CN3065_C2 4.7uF, CN3065_R1 1K8, CN3065_STDBY_LED1 LED, CN3965_C1 22uF, J1 Conn_01x07_Socket, J1 TYPE-C-31-M-12, J3 U.FL-R-SMT(01), J6 RFShield_OnePiece, U1 ATSHA204A-MAHDA-T, U1 MCP1525-TT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

Commit message: Add files via upload
Parts:
- added ATH20_C1: 100nF, Capacitor_SMD:C_0603_1608Metric, symbol Device:C
- added IC_ENS1: ~, AeonLabs_Sensors:ENS160 Gas Semsor, symbol AeonLabs_Sensors:ENS160_Gas_Sensor
- added U5: BMP280, AeonLabs_Sensors:XDCR_BMP280, symbol AeonLabs_Sensors:BMP280
- U1: footprint Package_SO:ATSHA204A Auth SOIC8 -> AeonLabs_IC:ATSHA204A-MAHDA-T UDFN-8
Connections:
- net 3V3: now also ATH20_C1.2, IC_ENS1.4 (VDD), IC_ENS1.5 (VDDIO), IC_ENS1.7 (CS), U5.2 (CSB), U5.6 (VDDIO), U5.8 (VDD)
- net GNDD: now also ATH20_C1.1, IC_ENS1.3 (MISO), IC_ENS1.8 (VSS), IC_ENS1.9 (VSS), U5.1 (GND), U5.5 (SDO), U5.7 (GND)
- net GPIO8_I2C_SDA: now also IC_ENS1.1 (SDA), U5.3 (SDI)
- net GPIO9_I2C_SCL: now also IC_ENS1.2 (SCL), U5.4 (SCK)
- no-connect marks 16 -> 17
Other:
- note added: "C02 Gas Sensor"
- moved on the sheet: IMU1, TMPR1, U1, U4, U6, VOLTAGE_REF_C1, VOLTAGE_REF_C2
